File: Hardware/Alvaro.kicad_pcb (KiCad board)
At the start: 2 copper layers, 17.8 x 33 mm, 27 parts, among them J2 01x02, J3 01x12, J4 01x12, J5 01x05, P1 USB_C_Receptacle_USB2.0, U1 ATmega32U4, X1 16MHz

Commit message: Updated to V1.5
Parts:
- added JP1: RAW, Jumper:SolderJumper-2_P1.3mm_Open_Pad1.0x1.5mm, F.Cu at (37.5, 25.2)
- moved G*** 2.35 mm to (29.9, 38.6)
- moved R6 0.65 mm to (27.7, 35.0)
- moved R3 0.40 mm to (35.2, 32.4)
- moved C10 0.40 mm to (35.2, 35.4)
- moved C8 0.38 mm to (26.0, 48.0)
- moved R1 0.35 mm to (32.2, 32.5)
- moved R5 0.35 mm to (32.2, 35.5)
- moved C3 0.34 mm to (35.0, 39.6)
- moved R4 0.30 mm to (30.7, 34.9)
Connections:
- J3 pad 1: VBUS -> Net-(J3-Pad1)
Routing:
- net /PF0: track 32.0 -> 28.7 mm
- net VBUS: track 37.7 -> 40.0 mm, vias 3 -> 4
- net Net-(J3-Pad1): track 0.00 -> 2.21 mm
- net /PF1: track 29.7 -> 28.5 mm
- net /PF6: track 11.6 -> 10.6 mm
- net /PF5: track 9.64 -> 8.66 mm
- net /RESET: track 27.4 -> 26.5 mm
- net VCC: track 47.4 -> 46.7 mm
- net /PF4: track 8.34 -> 7.82 mm
Other:
- board text added: "V1.5 Aria"
- board text removed: "V1.4 Aria"
